Commit message: perfectly work version
Signed-off-by: Spike <vergil1133@live.com>

File: urdf/husky.urdf (robot description, URDF)
Before this commit: robot husky_robot, 11 links, 10 joints
Links:
- link base_link: mass 33.455 -> 133.455

File: urdf/robotiq_85.urdf (robot description, URDF)
Before this commit: robot robotiq_arg2f_85_model, 11 links, 10 joints
Joints:
- joint finger_joint: limit lower=0 upper=0.8 effort=1000 velocity=2.0 -> lower=0 upper=0.8 effort=1000 velocity=4.0
- joint left_inner_finger_joint: limit lower=-0.8757 upper=0 effort=1000 velocity=2.0 -> lower=-0.8757 upper=0 effort=1000 velocity=4.0
- joint left_inner_knuckle_joint: limit lower=0 upper=0.8757 effort=1000 velocity=2.0 -> lower=0 upper=0.8757 effort=1000 velocity=4.0
- joint right_inner_finger_joint: limit lower=-0.8757 upper=0 effort=1000 velocity=2.0 -> lower=-0.8757 upper=0 effort=1000 velocity=4.0
- joint right_inner_knuckle_joint: limit lower=0 upper=0.8757 effort=1000 velocity=2.0 -> lower=0 upper=0.8757 effort=1000 velocity=4.0
- joint right_outer_knuckle_joint: limit lower=0 upper=0.81 effort=1000 velocity=2.0 -> lower=0 upper=0.81 effort=1000 velocity=4.0
