Commit message: updated
Signed-off-by: Spike <vergil1133@live.com>

File: urdf/ball_1/ball.urdf (robot description, URDF)
Before this commit: robot none, 1 links, 0 joints
Links:
- removed link none
- added link ball, mass 0; collision sphere radius=0.04; visual sphere radius=0.04

File: urdf/block/brick_0.3/brick.urdf (robot description, URDF)
Before this commit: robot none, 1 links, 0 joints
Links:
- link none: geometry collision box size=0.00000 0.00000 0.00000; visual mesh filename=cube.obj
